File: pcb/AVR_QuickLoader_PCB_V1.0/AVR_QuickLoader_PCB_V1.0.kicad_sch (KiCad schematic)
At the start: 15 parts, among them J1 USB_B, U1 CH340C, U2 ATmega328P-A, U3 ATmega328P-P, Y1 Crystal, Y2 Crystal

Commit message: added readme and started the pcb design routing
Parts:
- added C1: 100nF, Capacitor_SMD:C_0805_2012Metric_Pad1.18x1.45mm_HandSolder, symbol Device:C_Small
- added D1, D2, D3, D4, D5, D6: LED, LED_THT:LED_D3.0mm, symbol Device:LED
- added J2, J3: ICSP, Connector_PinHeader_2.54mm:PinHeader_2x03_P2.54mm_Vertical, symbol Connector_Generic:Conn_02x03_Odd_Even
- added R1, R2, R3, R4, R7, R8: 470, Resistor_SMD:R_0805_2012Metric_Pad1.20x1.40mm_HandSolder, symbol Device:R_Small_US
- added R5, R6: 10K, Resistor_SMD:R_0805_2012Metric_Pad1.20x1.40mm_HandSolder, symbol Device:R_Small_US
- renumbered C9 to C10, C1 to C2, C2 to C3, C3 to C4, C4 to C5, C5 to C6, C6 to C7, C7 to C8, C8 to C9
Connections:
- net +5V: now also C3.1, C4.1, J1.1 (VBUS), U1.16 (VCC), C1.1, D1.2 (A), D2.2 (A), D3.2 (A), D4.2 (A), D5.2 (A), D6.2 (A), J2.2 (Pin_2), J3.2 (Pin_2), R5.1, R6.1
- net GND: now also C1.2, J2.6 (Pin_6), J3.6 (Pin_6), R1.1
- net pUC_DTR: now also R5.2
- net pUC_OSC1: now also U2.7 (XTAL1/PB6)
- net pUC_OSC2: now also U2.8 (XTAL2/PB7)
- net pUC_RX: now also R7.1
- net pUC_TX: now also R8.1
- net tUC_DTR: now reaches U2.14 (PB2)
- net tUC_DTR: now also U3.1 (~{RESET}/PC6), J2.5 (Pin_5), J3.5 (Pin_5), R6.2
- net SPI_MOSI: now reaches U2.15 (PB3)
- net SPI_MOSI: now also U3.17 (PB3), J2.4 (Pin_4), J3.3 (Pin_3), R2.1
- net SPI_MISO: now reaches U2.16 (PB4)
- net SPI_MISO: now also U3.18 (PB4), J2.1 (Pin_1), J3.1 (Pin_1), R3.1
- net SPI_CLK: now reaches U2.17 (PB5)
- net SPI_CLK: now also U3.19 (PB5), J2.3 (Pin_3), J3.4 (Pin_4), R4.1
- net tUC_TX: now reaches U3.2 (PD0)
- net tUC_RX: now reaches U3.3 (PD1)
- new net: D2.1 (K), R2.2
- new net: D6.1 (K), R8.2
- new net: D4.1 (K), R4.2
- new net: D1.1 (K), R1.2
- new net: D5.1 (K), R7.2
- new net: D3.1 (K), R3.2
Other:
- note added: "Arduino ICSP"
- note added: "KNScore ICSP"
