File: pcb/AVR_QuickLoader_PCB_V1.0/_restore_backup_2026-06-08T15-51-57-227/AVR_QuickLoader_PCB_V1.0.kicad_sch (KiCad schematic)
At the start: 32 parts, among them J1 USB_B, J2 ICSP, J3 ICSP, U1 CH340C, U2 ATmega328P-A, U3 ATmega328P-P, Y1 Crystal, Y2 Crystal

Commit message: refactored the arrangement on the SCH file
Other:
- note added: "PROGRAMMER MCU"
- note added: "TARGET MCU"
- note removed: "PROGRAMMER MCU ICSP"
- note removed: "TARGET MCU ICSP"
- note removed: "USB TO TTL"
- moved on the sheet: C1, C10, C2, C3, C4, C5, C6, C7, C8, C9, D1, D2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
